Commit message: added the joints, head, and created scripts to easily run all things

File: description/robot.urdf.xacro (robot description, xacro)
@@ -2,3 +2,5 @@
 <robot xmlns:xacro="http://www.ros.org/wiki/xacro"  name="robot">
     <xacro:include filename="robot_core.xacro" />
+    <xacro:include filename="gazebo_control.xacro"/>
+    <xacro:include filename="robot_head.xacro"/>
 </robot>

File: description/robot_core.xacro (robot description, xacro)
@@ -17,5 +17,5 @@
         <color rgba="1 0 0 1"/>
     </material>
-     <material name="yellow">
+    <material name="yellow">
         <color rgba="1 1 0 1"/>
     </material>
@@ -47,4 +47,7 @@
         </xacro:inertial_box>
     </link>
+    <gazebo reference="chassis">
+        <material>Gazebo/Yellow</material>
+    </gazebo>
     <!-- LEFT WHEEL LINK -->
     <joint name="left_wheel_joint" type="continuous">
@@ -70,4 +73,7 @@
         </xacro:inertial_cylinder>
     </link>
+    <gazebo reference="left_wheel">
+        <material>Gazebo/Black</material>
+    </gazebo>
         <!-- RIGHT WHEEL LINK -->
     <joint name="right_wheel_joint" type="continuous">
@@ -93,4 +99,7 @@
         </xacro:inertial_cylinder>
     </link>
+    <gazebo reference="right_wheel">
+        <material>Gazebo/Black</material>
+    </gazebo>
     <!-- LEFT CASTER WHEEL LINK -->
     <joint name="left_caster_wheel_joint" type="fixed">
@@ -115,4 +124,9 @@
         </xacro:inertial_cylinder>
     </link>
+    <gazebo reference="left_caster_wheel">
+        <material>Gazebo/Black</material>
+        <mu1 value="0.001"/>
+        <mu2 value="0.001"/>
+    </gazebo>
         <!-- RIGHT CASTER WHEEL LINK -->
     <joint name="right_caster_wheel_joint" type="fixed">
@@ -137,3 +151,8 @@
         </xacro:inertial_cylinder>
     </link>
+    <gazebo reference="right_caster_wheel">
+        <material>Gazebo/Black</material>
+        <mu1 value="0.001"/>
+        <mu2 value="0.001"/>
+    </gazebo>
 </robot>

Commit message: Added lidar xacro file

File: description/robot.urdf.xacro (robot description, xacro)
@@ -4,3 +4,4 @@
     <xacro:include filename="gazebo_control.xacro"/>
     <xacro:include filename="robot_head.xacro"/>
+    <xacro:include filename="lidar.xacro"/>
 </robot>

File: description/robot_head.xacro (robot description, xacro)
@@ -1,5 +1,5 @@
 <?xml version="1.0"?>
 <robot xmlns:xacro="http://www.ros.org/wiki/xacro" >
-    <joint name="head_joint" type="revolute">
+    <joint name="head_joint" type="fixed">
         <parent link="chassis"/>
         <child link="head"/>
